Commit message: Corrected base_link->laser transform
Not necessary for other robots, this was a purely personal change

File: launch/UGV.urdf (robot description, URDF)
Before this commit: robot UGV, 4 links, 3 joints
Joints:
- joint base_to_laser: origin xyz=0.1524 0 0.2032 rpy=0 0 3.14159265359 -> xyz=0.149225 0 0.1778 rpy=0 0 3.14159265359
